Commit message: fix: align SO101 MoveIt and ros2_control configuration

File: src/so101_follower_description/urdf/so101_follower.urdf.xacro (robot description, xacro)
@@ -3,5 +3,8 @@
 <!-- Onshape https://cad.onshape.com/documents/7715cc284bb430fe6dab4ffd/w/4fd0791b683777b02f8d975a/e/826c553ede3b7592eb9ca800 -->
 <robot name="so101_follower" xmlns:xacro="http://www.ros.org/wiki/xacro">
-  <xacro:include filename="$(find so101_hw_interface)/urdf/so101_follower.urdf" />
+  <xacro:arg name="use_fake_hardware" default="false" />
+  <xacro:unless value="$(arg use_fake_hardware)">
+    <xacro:include filename="$(find so101_hw_interface)/urdf/so101_follower.urdf" />
+  </xacro:unless>
   <!-- World Link -->
   <link name="world"/>

File: src/so101_follower_moveit/config/so101_follower.ros2_control.xacro (robot description, xacro)
@@ -18,5 +18,4 @@
                   <param name="initial_value">${load_yaml(initial_positions_file)['initial_positions']['shoulder_pan'] if initial_positions_file != '/dev/null' else '0.0'}</param>
                 </state_interface>
-                <state_interface name="velocity"/>
             </joint>
             <joint name="shoulder_lift">
@@ -25,5 +24,4 @@
                     <param name="initial_value">${load_yaml(initial_positions_file)['initial_positions']['shoulder_lift'] if initial_positions_file != '/dev/null' else '0.0'}</param>
                 </state_interface>
-                <state_interface name="velocity"/>
             </joint>
             <joint name="elbow_flex">
@@ -32,5 +30,4 @@
                     <param name="initial_value">${load_yaml(initial_positions_file)['initial_positions']['elbow_flex'] if initial_positions_file != '/dev/null' else '0.0'}</param>
                 </state_interface>
-                <state_interface name="velocity"/>
             </joint>
             <joint name="wrist_flex">
@@ -39,5 +36,4 @@
                     <param name="initial_value">${load_yaml(initial_positions_file)['initial_positions']['wrist_flex'] if initial_positions_file != '/dev/null' else '0.0'}</param>
                 </state_interface>
-                <state_interface name="velocity"/>
             </joint>
             <joint name="wrist_roll">
@@ -46,22 +42,10 @@
                     <param name="initial_value">${load_yaml(initial_positions_file)['initial_positions']['wrist_roll'] if initial_positions_file != '/dev/null' else '0.0'}</param>
                 </state_interface>
-                <state_interface name="velocity"/>
             </joint>
-            <joint name="wrist_pitch">
-                <command_interface name="position"/>
-                <state_interface name="position"/>
-                <state_interface name="velocity"/>
-            </joint>
-            <joint name="wrist_yaw">
-                <command_interface name="position"/>
-                <state_interface name="position"/>
-                <state_interface name="velocity"/>
-            </joint>
-            <joint name="gripper_jaw">
+            <joint name="gripper">
                 <command_interface name="position"/>
                 <state_interface name="position">
                     <param name="initial_value">${load_yaml(initial_positions_file)['initial_positions']['gripper'] if initial_positions_file != '/dev/null' else '0.0'}</param>
                 </state_interface>
-                <state_interface name="velocity"/>
             </joint>
         </ros2_control>

File: src/so101_follower_moveit/config/so101_follower.urdf.xacro (robot description, xacro)
@@ -10,6 +10,3 @@
         <xacro:so101_follower_ros2_control name="FakeSystem" initial_positions_file="$(find so101_follower_moveit)/config/initial_positions.yaml"/>
     </xacro:if>
-    <xacro:unless value="$(arg use_fake_hardware)">
-        <xacro:so101_follower_ros2_control name="so101_follower"/>
-    </xacro:unless>
 </robot>

Commit message: feat: add nominal TCP and robot TF publishing

File: src/so101_follower_description/urdf/so101_follower.urdf.xacro (robot description, xacro)
@@ -294,4 +294,12 @@
     </collision>
   </link>
+  <!-- CAD-derived nominal grasp TCP at gripper q_ref=0, not physically calibrated.
+       This fixed frame does not track the grasp midpoint at other openings. -->
+  <link name="tcp_link"/>
+  <joint name="gripper_to_tcp" type="fixed">
+    <parent link="gripper_link"/>
+    <child link="tcp_link"/>
+    <origin xyz="0.000150 -0.000159 -0.074598" rpy="0 0 0"/>
+  </joint>
   <!-- Link jaw -->
   <link name="jaw_link">
